File: Term.sch (KiCad schematic (older format))
At the start: 21 parts, among them J1 JACK_TRS, P1 UART0, SW1 RESET, SW2 FLASH, SW3 SW_SPST, U1 LM1117-3.3, U2 ESP-12F

Commit message: v0.1 - Connection and deep sleep work.
Parts:
- R1: value 10M -> 100k
- R2, R3: value 33k -> 22k
- R4: value 10k -> 2k2
Connections:
- wire segments 44 -> 47
Other:
- moved on the sheet: C4, D1, R1, R4
Changed lines of the file:
@@
 Text Label 6650 3200 0    60   ~ 0
 ~RST
-Wire Wire Line
-	5350 3400 7150 3400
 $Comp
 L +3V3 #PWR04
 U 1 1 590235A0
-P 5350 3400
-F 0 "#PWR04" H 5350 3250 50  0001 C CNN
-F 1 "+3V3" H 5350 3540 50  0000 C CNN
-F 2 "" H 5350 3400 50  0000 C CNN
-F 3 "" H 5350 3400 50  0000 C CNN
-	1    5350 3400
+P 5100 3400
+F 0 "#PWR04" H 5100 3250 50  0001 C CNN
+F 1 "+3V3" H 5100 3540 50  0000 C CNN
+F 2 "" H 5100 3400 50  0000 C CNN
+F 3 "" H 5100 3400 50  0000 C CNN
+	1    5100 3400
 	1    0    0    -1
 $EndComp
@@
 L R R1
 U 1 1 590235C2
-P 5500 3550
-F 0 "R1" V 5580 3550 50  0000 C CNN
-F 1 "10M" V 5500 3550 50  0000 C CNN
-F 2 "Resistors_THT:R_Axial_DIN0207_L6.3mm_D2.5mm_P7.62mm_Horizontal" V 5430 3550 50  0001 C CNN
-F 3 "" H 5500 3550 50  0000 C CNN
-	1    5500 3550
-	1    0    0    -1
+P 5500 3400
+F 0 "R1" V 5580 3400 50  0000 C CNN
+F 1 "100k" V 5500 3400 50  0000 C CNN
+F 2 "Resistors_THT:R_Axial_DIN0207_L6.3mm_D2.5mm_P7.62mm_Horizontal" V 5430 3400 50  0001 C CNN
+F 3 "" H 5500 3400 50  0000 C CNN
+	1    5500 3400
+	0    1    1    0
 $EndComp
 $Comp
 L C C4
 U 1 1 59023831
-P 5500 3850
-F 0 "C4" H 5525 3950 50  0000 L CNN
-F 1 "10n" H 5525 3750 50  0000 L CNN
-F 2 "Capacitors_THT:C_Disc_D4.3mm_W1.9mm_P5.00mm" H 5538 3700 50  0001 C CNN
-F 3 "" H 5500 3850 50  0000 C CNN
-	1    5500 3850
+P 6000 3650
+F 0 "C4" H 6025 3750 50  0000 L CNN
+F 1 "10n" H 6025 3550 50  0000 L CNN
+F 2 "Capacitors_THT:C_Disc_D4.3mm_W1.9mm_P5.00mm" H 6038 3500 50  0001 C CNN
+F 3 "" H 6000 3650 50  0000 C CNN
+	1    6000 3650
 	1    0    0    -1
 $EndComp
@@
 L GND #PWR05
 U 1 1 59023874
-P 5500 4050
-F 0 "#PWR05" H 5500 3800 50  0001 C CNN
-F 1 "GND" H 5500 3900 50  0000 C CNN
-F 2 "" H 5500 4050 50  0000 C CNN
-F 3 "" H 5500 4050 50  0000 C CNN
-	1    5500 4050
-	1    0    0    -1
-$EndComp
-Wire Wire Line
-	5500 4000 5500 4050
+P 6000 3850
+F 0 "#PWR05" H 6000 3600 50  0001 C CNN
+F 1 "GND" H 6000 3700 50  0000 C CNN
+F 2 "" H 6000 3850 50  0000 C CNN
+F 3 "" H 6000 3850 50  0000 C CNN
+	1    6000 3850
+	1    0    0    -1
+$EndComp
+Wire Wire Line
+	6000 3800 6000 3850
 $Comp
 L +3V3 #PWR06
@@
 P 6400 2700
 F 0 "R2" V 6480 2700 50  0000 C CNN
-F 1 "33k" V 6400 2700 50  0000 C CNN
+F 1 "22k" V 6400 2700 50  0000 C CNN
 F 2 "Resistors_THT:R_Axial_DIN0207_L6.3mm_D2.5mm_P7.62mm_Horizontal" V 6330 2700 50  0001 C CNN
 F 3 "" H 6400 2700 50  0000 C CNN
@@
 P 9100 3450
 F 0 "R3" V 9180 3450 50  0000 C CNN
-F 1 "33k" V 9100 3450 50  0000 C CNN
+F 1 "22k" V 9100 3450 50  0000 C CNN
 F 2 "Resistors_THT:R_Axial_DIN0207_L6.3mm_D2.5mm_P7.62mm_Horizontal" V 9030 3450 50  0001 C CNN
 F 3 "" H 9100 3450 50  0000 C CNN
@@
 Wire Wire Line
 	9600 3600 9600 3600
-Wire Wire Line
-	8250 3500 8950 3500
 Text Label 2300 2250 0    60   ~ 0
 TH1
@@
 NoConn ~ 7850 4250
 NoConn ~ 7950 4250
-NoConn ~ 8250 3800
 NoConn ~ 8250 3700
 NoConn ~ 8250 3400
@@
 Wire Wire Line
 	8350 2750 8400 2750
-NoConn ~ 7150 3800
 NoConn ~ 7150 3700
 Wire Wire Line
@@
 $EndComp
 Connection ~ 3200 2100
-Connection ~ 5500 3400
 Connection ~ 6900 3900
 Wire Wire Line
 	2900 1450 3650 1450
-Text Label 8950 3500 2    60   ~ 0
+Text Label 8850 3500 2    60   ~ 0
 SENSE_PWR
 Text Label 3650 1450 2    60   ~ 0
@@
 L LED_ALT D1
 U 1 1 59036B62
+P 4550 6400
+F 0 "D1" H 4550 6500 50  0000 C CNN
+F 1 "LED_ALT" H 4550 6300 50  0000 C CNN
+F 2 "LEDs:LED_D5.0mm" H 4550 6400 50  0001 C CNN
+F 3 "" H 4550 6400 50  0000 C CNN
+	1    4550 6400
+	1    0    0    -1
+$EndComp
+Wire Wire Line
+	4850 6000 4850 6050
+$Comp
+L R R4
+U 1 1 59036D6C
 P 4850 6200
-F 0 "D1" H 4850 6300 50  0000 C CNN
-F 1 "LED_ALT" H 4850 6100 50  0000 C CNN
-F 2 "LEDs:LED_D5.0mm" H 4850 6200 50  0001 C CNN
+F 0 "R4" V 4930 6200 50  0000 C CNN
+F 1 "2k2" V 4850 6200 50  0000 C CNN
+F 2 "Resistors_THT:R_Axial_DIN0207_L6.3mm_D2.5mm_P7.62mm_Horizontal" V 4780 6200 50  0001 C CNN
 F 3 "" H 4850 6200 50  0000 C CNN
 	1    4850 6200
-	0    -1   -1   0
-$EndComp
-Wire Wire Line
-	4850 6000 4850 6050
-$Comp
-L R R4
-U 1 1 59036D6C
-P 4550 6400
-F 0 "R4" V 4630 6400 50  0000 C CNN
-F 1 "10k" V 4550 6400 50  0000 C CNN
-F 2 "Resistors_THT:R_Axial_DIN0207_L6.3mm_D2.5mm_P7.62mm_Horizontal" V 4480 6400 50  0001 C CNN
-F 3 "" H 4550 6400 50  0000 C CNN
-	1    4550 6400
-	0    1    1    0
+	-1   0    0    1
 $EndComp
 Wire Wire Line
@@
 Connection ~ 4150 6400
 NoConn ~ 7150 3600
+Wire Wire Line
+	6000 3500 6000 3400
+Connection ~ 6000 3400
+Wire Wire Line
+	5100 3400 5350 3400
+Wire Wire Line
+	5650 3400 7150 3400
+NoConn ~ 8250 3500
+Wire Wire Line
+	8250 3500 8850 3500
+NoConn ~ 7150 3800
+Wire Wire Line
+	8250 3900 8250 3800
 $EndSCHEMATC
